Commit message: Add Wheeled foot directory

File: TRON_description/WF_TRON1A/urdf/WF_TRON.urdf (robot description, URDF)
Before this commit: robot wheel_TRON, 10 links, 9 joints
Links:
- removed link limx_imu
Joints:
- removed joint limx_imu_joint

Commit message: add GOAT base_env, cfg

File: TRON_description/WF_TRON1A/urdf/WF_TRON.urdf (robot description, URDF)
Before this commit: robot wheel_TRON, 9 links, 8 joints
Links:
- removed link abad_L_Link
- removed link abad_R_Link
- removed link knee_L_Link
- removed link knee_R_Link
- added link calf_L_Link, mass 1.49; collision cylinder length=0.26 radius=0.015; visual mesh filename=../meshes/calf_L_Link.STL
- added link calf_R_Link, mass 1.49; collision cylinder length=0.26 radius=0.015; visual mesh filename=../meshes/calf_R_Link.STL
- added link thigh_L_Link, mass 2.3; collision cylinder length=0.15 radius=0.035; visual mesh filename=../meshes/thigh_L_Link.STL
- added link thigh_R_Link, mass 2.30; collision cylinder length=0.15 radius=0.035; visual mesh filename=../meshes/thigh_R_Link.STL
- link hip_L_Link: mass 2.3 -> 1.469; geometry collision cylinder length=0.05 radius=0.05; visual mesh filename=../meshes/hip_L_Link.STL
- link hip_R_Link: mass 2.30 -> 1.469; geometry collision cylinder length=0.05 radius=0.05; visual mesh filename=../meshes/hip_R_Link.STL
Joints:
- removed joint abad_L_Joint
- removed joint abad_R_Joint
- added joint thigh_L_Joint: type revolute, parent hip_L_Link, child thigh_L_Link, origin xyz=-0.077 0.02050 0 rpy=0 0 0, axis 0 1 0, limit lower=-1.012291 upper=1.396263 effort=80.0 velocity=15.0
- added joint thigh_R_Joint: type revolute, parent hip_R_Link, child thigh_R_Link, origin xyz=-0.077 -0.02050 0 rpy=0 0 0, axis 0 -1 0, limit lower=-1.396263 upper=1.012291 effort=80.0 velocity=15.0
- joint hip_L_Joint: axis 0 1 0 -> 1 0 0; limit lower=-1.012291 upper=1.396263 effort=80.0 velocity=15.0 -> lower=-0.38397 upper=1.39626 effort=80.0 velocity=15.0; origin xyz=-0.077 0.02050 0 rpy=0 0 0 -> xyz=55.56E-03 105E-03 -260.2E-03 rpy=0 0 0; parent abad_L_Link -> base_Link
- joint hip_R_Joint: axis 0 -1 0 -> 1 0 0; limit lower=-1.396263 upper=1.012291 effort=80.0 velocity=15.0 -> lower=-1.39626 upper=0.38397 effort=80.0 velocity=15.0; origin xyz=-0.077 -0.02050 0 rpy=0 0 0 -> xyz=55.56E-03 -105E-03 -260.2E-03 rpy=0 0 0; parent abad_R_Link -> base_Link
- joint knee_L_Joint: child knee_L_Link -> calf_L_Link; parent hip_L_Link -> thigh_L_Link
- joint knee_R_Joint: child knee_R_Link -> calf_R_Link; parent hip_R_Link -> thigh_R_Link
- joint wheel_L_Joint: parent knee_L_Link -> calf_L_Link
- joint wheel_R_Joint: parent knee_R_Link -> calf_R_Link
