Commit message: edit urdf

File: Realworld/src/goat_control/assets/WF_GOAT/urdf/WF_GOAT.urdf (robot description, URDF)
Before this commit: robot wheel_TRON, 9 links, 8 joints
Links:
- link base_Link: geometry collision box size=0.27 0.26 0.19; visual mesh filename=../meshes/base_Link.stl
- link calf_L_Link: geometry collision cylinder length=0.26 radius=0.015; visual mesh filename=../meshes/calf_L_Link.stl
- link calf_R_Link: geometry collision cylinder length=0.26 radius=0.015; visual mesh filename=../meshes/calf_R_Link.stl
- link hip_L_Link: geometry collision cylinder length=0.05 radius=0.05; visual mesh filename=../meshes/hip_L_Link.stl
- link hip_R_Link: geometry collision cylinder length=0.05 radius=0.05; visual mesh filename=../meshes/hip_R_Link.stl
- link thigh_L_Link: geometry collision cylinder length=0.15 radius=0.035; visual mesh filename=../meshes/thigh_L_Link.stl
- link thigh_R_Link: geometry collision cylinder length=0.15 radius=0.035; visual mesh filename=../meshes/thigh_R_Link.stl
- link wheel_L_Link: geometry collision cylinder length=0.05 radius=0.127; visual mesh filename=../meshes/wheel_L_Link.stl
- link wheel_R_Link: geometry collision cylinder length=0.05 radius=0.127; visual mesh filename=../meshes/wheel_R_Link.stl
Joints:
- joint knee_L_Joint: limit lower=0.0 upper=1.15192 effort=4.5 velocity=15 -> lower=0.0 upper=1.75192 effort=4.5 velocity=15; origin xyz=0 11.5E-03 -205E-03 rpy=0 0 0 -> xyz=0 18E-03 -205E-03 rpy=0 0 0
- joint knee_R_Joint: limit lower=-1.15192 upper=0.0 effort=4.5 velocity=15 -> lower=-1.75192 upper=0.0 effort=4.5 velocity=15; origin xyz=0 11.5E-03 -205E-03 rpy=0 0 0 -> xyz=0 -18E-03 -205E-03 rpy=0 0 0
- joint wheel_R_Joint: origin xyz=0 16.555E-03 -200E-03 rpy=0 0 0 -> xyz=0 -16.555E-03 -200E-03 rpy=0 0 0

File: lib/assets/GOAT/WF_GOAT/urdf/WF_GOAT.urdf (robot description, URDF)
Before this commit: robot wheel_TRON, 9 links, 8 joints
Links:
- link base_Link: geometry collision box size=0.27 0.26 0.19; visual mesh filename=../meshes/base_Link.stl
- link calf_L_Link: geometry collision cylinder length=0.26 radius=0.015; visual mesh filename=../meshes/calf_L_Link.stl
- link calf_R_Link: geometry collision cylinder length=0.26 radius=0.015; visual mesh filename=../meshes/calf_R_Link.stl
- link hip_L_Link: geometry collision cylinder length=0.05 radius=0.05; visual mesh filename=../meshes/hip_L_Link.stl
- link hip_R_Link: geometry collision cylinder length=0.05 radius=0.05; visual mesh filename=../meshes/hip_R_Link.stl
- link thigh_L_Link: geometry collision cylinder length=0.15 radius=0.035; visual mesh filename=../meshes/thigh_L_Link.stl
- link thigh_R_Link: geometry collision cylinder length=0.15 radius=0.035; visual mesh filename=../meshes/thigh_R_Link.stl
- link wheel_L_Link: geometry collision cylinder length=0.05 radius=0.127; visual mesh filename=../meshes/wheel_L_Link.stl
- link wheel_R_Link: geometry collision cylinder length=0.05 radius=0.127; visual mesh filename=../meshes/wheel_R_Link.stl
