Commit message: change screw axis

File: lib/assets/GOAT/WF_GOAT/urdf/WF_GOAT.urdf (robot description, URDF)
Before this commit: robot wheel_TRON, 9 links, 8 joints
Joints:
- joint hip_L_Joint: axis 1 0 0 -> -1 0 0
- joint knee_R_Joint: axis 0 1 0 -> 0 -1 0
- joint thigh_R_Joint: axis 0 -1 0 -> 0 1 0

Commit message: match screw axis to real motor axis

File: lib/assets/GOAT/WF_GOAT/urdf/WF_GOAT.urdf (robot description, URDF)
Before this commit: robot wheel_TRON, 9 links, 8 joints
Joints:
- joint hip_L_Joint: limit lower=-0.38397 upper=1.39626 effort=80.0 velocity=15.0 -> lower=-0.38397 upper=1.39626 effort=4.5 velocity=15.0
- joint hip_R_Joint: axis 1 0 0 -> -1 0 0; limit lower=-1.39626 upper=0.38397 effort=80.0 velocity=15.0 -> lower=-1.39626 upper=0.38397 effort=4.5 velocity=15.0
- joint knee_L_Joint: limit lower=-0.872665 upper=1.361357 effort=80 velocity=15 -> lower=-0.872665 upper=1.361357 effort=4.5 velocity=15
- joint knee_R_Joint: axis 0 -1 0 -> 0 1 0; limit lower=-1.361357 upper=0.872665 effort=80 velocity=15 -> lower=-1.361357 upper=0.872665 effort=4.5 velocity=15
- joint thigh_L_Joint: limit lower=-1.012291 upper=1.396263 effort=80.0 velocity=15.0 -> lower=-1.012291 upper=1.396263 effort=4.5 velocity=15.0
- joint thigh_R_Joint: axis 0 1 0 -> 0 -1 0; limit lower=-1.396263 upper=1.012291 effort=80.0 velocity=15.0 -> lower=-1.396263 upper=1.012291 effort=4.5 velocity=15.0
- joint wheel_L_Joint: axis 0 1 0 -> 0 -1 0; limit lower=-1000000 upper=1000000 effort=40 velocity=40 -> lower=-1000000 upper=1000000 effort=2.5 velocity=40
- joint wheel_R_Joint: limit lower=-1000000 upper=1000000 effort=40 velocity=40 -> lower=-1000000 upper=1000000 effort=2.5 velocity=40

Commit message: change joint limits

File: lib/assets/GOAT/WF_GOAT/urdf/WF_GOAT.urdf (robot description, URDF)
Before this commit: robot wheel_TRON, 9 links, 8 joints
Joints:
- joint hip_L_Joint: limit lower=-0.38397 upper=1.39626 effort=4.5 velocity=15.0 -> lower=-2.05949 upper=1.09956 effort=4.5 velocity=15.0
- joint hip_R_Joint: limit lower=-1.39626 upper=0.38397 effort=4.5 velocity=15.0 -> lower=-1.09956 upper=2.05949 effort=4.5 velocity=15.0
- joint knee_L_Joint: limit lower=-0.872665 upper=1.361357 effort=4.5 velocity=15 -> lower=0.0 upper=1.15192 effort=4.5 velocity=15
- joint knee_R_Joint: limit lower=-1.361357 upper=0.872665 effort=4.5 velocity=15 -> lower=-1.15192 upper=0.0 effort=4.5 velocity=15
- joint thigh_L_Joint: limit lower=-1.012291 upper=1.396263 effort=4.5 velocity=15.0 -> lower=-0.593412 upper=0.314159 effort=4.5 velocity=15.0
- joint thigh_R_Joint: limit lower=-1.396263 upper=1.012291 effort=4.5 velocity=15.0 -> lower=-0.314159 upper=0.593412 effort=4.5 velocity=15.0

Commit message: change thigh joint limit

File: lib/assets/GOAT/WF_GOAT/urdf/WF_GOAT.urdf (robot description, URDF)
Before this commit: robot wheel_TRON, 9 links, 8 joints
Joints:
- joint thigh_L_Joint: limit lower=-0.593412 upper=0.314159 effort=4.5 velocity=15.0 -> lower=-0.593412 upper=1.88496 effort=4.5 velocity=15.0
- joint thigh_R_Joint: limit lower=-0.314159 upper=0.593412 effort=4.5 velocity=15.0 -> lower=-1.88496 upper=0.593412 effort=4.5 velocity=15.0

Commit message: feat

File: lib/assets/GOAT/WF_GOAT/urdf/WF_GOAT.urdf (robot description, URDF)
Before this commit: robot wheel_TRON, 9 links, 8 joints
Joints:
- joint knee_R_Joint: origin xyz=0 11.5E-03 -205E-03 rpy=0 0 0 -> xyz=0 -11.5E-03 -205E-03 rpy=0 0 0
- joint wheel_R_Joint: origin xyz=0 16.555E-03 -200E-03 rpy=0 0 0 -> xyz=0 -16.555E-03 -200E-03 rpy=0 0 0

Commit message: feat

File: lib/assets/GOAT/WF_GOAT/urdf/WF_GOAT.urdf (robot description, URDF)
Before this commit: robot wheel_TRON, 9 links, 8 joints
Joints:
- joint knee_L_Joint: limit lower=0.0 upper=1.15192 effort=4.5 velocity=15 -> lower=0.0 upper=1.75192 effort=4.5 velocity=15; origin xyz=0 11.5E-03 -205E-03 rpy=0 0 0 -> xyz=0 18E-03 -205E-03 rpy=0 0 0
- joint knee_R_Joint: limit lower=-1.15192 upper=0.0 effort=4.5 velocity=15 -> lower=-1.75192 upper=0.0 effort=4.5 velocity=15; origin xyz=0 -11.5E-03 -205E-03 rpy=0 0 0 -> xyz=0 -18E-03 -205E-03 rpy=0 0 0

Commit message: feat : simulation visualization with rvizwq

File: lib/assets/GOAT/WF_GOAT/urdf/WF_GOAT.urdf (robot description, URDF)
Before this commit: robot wheel_TRON, 9 links, 8 joints
Links:
- link base_Link: geometry collision box size=0.27 0.26 0.19; visual mesh filename=../meshes/base_Link.STL
- link calf_L_Link: geometry collision cylinder length=0.26 radius=0.015; visual mesh filename=../meshes/calf_L_Link.STL
- link calf_R_Link: geometry collision cylinder length=0.26 radius=0.015; visual mesh filename=../meshes/calf_R_Link.STL
- link hip_L_Link: geometry collision cylinder length=0.05 radius=0.05; visual mesh filename=../meshes/hip_L_Link.STL
- link hip_R_Link: geometry collision cylinder length=0.05 radius=0.05; visual mesh filename=../meshes/hip_R_Link.STL
- link thigh_L_Link: geometry collision cylinder length=0.15 radius=0.035; visual mesh filename=../meshes/thigh_L_Link.STL
- link thigh_R_Link: geometry collision cylinder length=0.15 radius=0.035; visual mesh filename=../meshes/thigh_R_Link.STL
- link wheel_L_Link: geometry collision cylinder length=0.05 radius=0.127; visual mesh filename=../meshes/wheel_L_Link.STL
- link wheel_R_Link: geometry collision cylinder length=0.05 radius=0.127; visual mesh filename=../meshes/wheel_R_Link.STL

Commit message: feat: adding inertia tensor

File: lib/assets/GOAT/WF_GOAT/urdf/WF_GOAT.urdf (robot description, URDF)
Before this commit: robot wheel_TRON, 9 links, 8 joints
Links:
- link base_Link: mass 9.585 -> 2.818
- link calf_L_Link: mass 1.49 -> 0.287
- link calf_R_Link: mass 1.49 -> 0.287
- link hip_L_Link: mass 1.469 -> 0.32
- link hip_R_Link: mass 1.469 -> 0.32
- link thigh_L_Link: mass 2.3 -> 0.429
- link thigh_R_Link: mass 2.30 -> 0.429
- link wheel_L_Link: mass 1.08 -> 0.212
- link wheel_R_Link: mass 1.08 -> 0.212

Commit message: stl file mapping

File: lib/assets/GOAT/WF_GOAT/urdf/WF_GOAT.urdf (robot description, URDF)
Before this commit: robot wheel_TRON, 9 links, 8 joints
Links:
- link base_Link: geometry collision box size=0.27 0.26 0.19; visual mesh filename=../meshes/base_Link.stl
- link calf_L_Link: geometry collision cylinder length=0.26 radius=0.015; visual mesh filename=../meshes/calf_L_Link.stl
- link calf_R_Link: geometry collision cylinder length=0.26 radius=0.015; visual mesh filename=../meshes/calf_R_Link.stl
- link hip_L_Link: geometry collision cylinder length=0.05 radius=0.05; visual mesh filename=../meshes/hip_L_Link.stl
- link hip_R_Link: geometry collision cylinder length=0.05 radius=0.05; visual mesh filename=../meshes/hip_R_Link.stl
- link thigh_L_Link: geometry collision cylinder length=0.15 radius=0.035; visual mesh filename=../meshes/thigh_L_Link.stl
- link thigh_R_Link: geometry collision cylinder length=0.15 radius=0.035; visual mesh filename=../meshes/thigh_R_Link.stl
- link wheel_L_Link: geometry collision cylinder length=0.05 radius=0.127; visual mesh filename=../meshes/wheel_L_Link.stl
- link wheel_R_Link: geometry collision cylinder length=0.05 radius=0.127; visual mesh filename=../meshes/wheel_R_Link.stl

Commit message: feat : urdf collision rejion fix

File: lib/assets/GOAT/WF_GOAT/urdf/WF_GOAT.urdf (robot description, URDF)
Before this commit: robot wheel_TRON, 9 links, 8 joints
Links:
- link hip_L_Link: geometry collision cylinder length=48E-03 radius=43.5E-03; visual mesh filename=../meshes/hip_L_Link.STL
- link hip_R_Link: geometry collision cylinder length=48E-03 radius=43.5E-03; visual mesh filename=../meshes/hip_R_Link.STL
- link thigh_L_Link: geometry collision cylinder length=266E-03 radius=41E-03; visual mesh filename=../meshes/thigh_L_Link.STL
- link thigh_R_Link: geometry collision cylinder length=266E-03 radius=41E-03; visual mesh filename=../meshes/thigh_R_Link.STL

Commit message: feat: urdf collision region setting

File: lib/assets/GOAT/WF_GOAT/urdf/WF_GOAT.urdf (robot description, URDF)
Before this commit: robot wheel_TRON, 9 links, 8 joints
Links:
- link base_Link: mass 9.585 -> 2.818; geometry collision box size=0.214 0.200 0.190; visual mesh filename=../meshes/base_Link.STL
- link calf_L_Link: mass 1.49 -> 0.287; geometry collision cylinder length=233E-03 radius=32.5E-03; visual mesh filename=../meshes/calf_L_Link.STL
- link calf_R_Link: mass 1.49 -> 0.287; geometry collision cylinder length=233E-03 radius=32.5E-03; visual mesh filename=../meshes/calf_R_Link.STL
- link hip_L_Link: mass 1.469 -> 0.32; geometry collision cylinder length=48E-03 radius=43.5E-03; visual mesh filename=../meshes/hip_L_Link.STL
- link hip_R_Link: mass 1.469 -> 0.32; geometry collision cylinder length=48E-03 radius=43.5E-03; visual mesh filename=../meshes/hip_R_Link.STL
- link thigh_L_Link: mass 2.3 -> 0.429; geometry collision cylinder length=266E-03 radius=41E-03; visual mesh filename=../meshes/thigh_L_Link.STL
- link thigh_R_Link: mass 2.30 -> 0.429; geometry collision cylinder length=266E-03 radius=41E-03; visual mesh filename=../meshes/thigh_R_Link.STL
- link wheel_L_Link: mass 1.08 -> 0.212; geometry collision cylinder length=32E-03 radius=73E-03; visual mesh filename=../meshes/wheel_L_Link.STL
- link wheel_R_Link: mass 1.08 -> 0.212; geometry collision cylinder length=32E-03 radius=73E-03; visual mesh filename=../meshes/wheel_R_Link.STL

Commit message: feat : wheel collision region fix

File: lib/assets/GOAT/WF_GOAT/urdf/WF_GOAT.urdf (robot description, URDF)
Before this commit: robot wheel_TRON, 9 links, 8 joints
Links:
- link wheel_L_Link: geometry collision cylinder length=32E-03 radius=72.75E-03; visual mesh filename=../meshes/wheel_L_Link.STL
- link wheel_R_Link: geometry collision cylinder length=32E-03 radius=72.75E-03; visual mesh filename=../meshes/wheel_R_Link.STL

Commit message: real2sim

File: lib/assets/GOAT/WF_GOAT/urdf/WF_GOAT.urdf (robot description, URDF)
Before this commit: robot wheel_TRON, 9 links, 8 joints
Links:
- link base_Link: geometry collision box size=0.214 0.200 0.190; visual mesh filename=../meshes/base_Link.stl
- link calf_L_Link: geometry collision cylinder length=233E-03 radius=32.5E-03; visual mesh filename=../meshes/calf_L_Link.stl
- link calf_R_Link: geometry collision cylinder length=233E-03 radius=32.5E-03; visual mesh filename=../meshes/calf_R_Link.stl
- link hip_L_Link: geometry collision cylinder length=48E-03 radius=43.5E-03; visual mesh filename=../meshes/hip_L_Link.stl
- link hip_R_Link: geometry collision cylinder length=48E-03 radius=43.5E-03; visual mesh filename=../meshes/hip_R_Link.stl
- link thigh_L_Link: geometry collision cylinder length=266E-03 radius=41E-03; visual mesh filename=../meshes/thigh_L_Link.stl
- link thigh_R_Link: geometry collision cylinder length=266E-03 radius=41E-03; visual mesh filename=../meshes/thigh_R_Link.stl
- link wheel_L_Link: geometry collision cylinder length=32E-03 radius=72.75E-03; visual mesh filename=../meshes/wheel_L_Link.stl
- link wheel_R_Link: geometry collision cylinder length=32E-03 radius=72.75E-03; visual mesh filename=../meshes/wheel_R_Link.stl
Joints:
- joint wheel_L_Joint: axis 0 -1 0 -> 0 1 0
- joint wheel_R_Joint: axis 0 1 0 -> 0 -1 0

Commit message: edir knee limit

File: lib/assets/GOAT/WF_GOAT/urdf/WF_GOAT.urdf (robot description, URDF)
Before this commit: robot wheel_GOAT, 9 links, 8 joints
Joints:
- joint knee_L_Joint: limit lower=0.0 upper=1.75192 effort=4.5 velocity=15 -> lower=-0.523599 upper=1.75192 effort=4.5 velocity=15
- joint knee_R_Joint: limit lower=-1.75192 upper=0.0 effort=4.5 velocity=15 -> lower=-1.75192 upper=0.523599 effort=4.5 velocity=15

Commit message: apply GOAT velocity limit

File: lib/assets/GOAT/WF_GOAT/urdf/WF_GOAT.urdf (robot description, URDF)
Before this commit: robot wheel_GOAT, 9 links, 8 joints
Joints:
- joint hip_L_Joint: limit lower=-2.05949 upper=1.09956 effort=4.5 velocity=15.0 -> lower=-2.05949 upper=1.09956 effort=4.5 velocity=33.5
- joint hip_R_Joint: limit lower=-1.09956 upper=2.05949 effort=4.5 velocity=15.0 -> lower=-1.09956 upper=2.05949 effort=4.5 velocity=33.5
- joint knee_L_Joint: limit lower=-0.523599 upper=1.75192 effort=4.5 velocity=15 -> lower=-0.523599 upper=1.75192 effort=4.5 velocity=33.5
- joint knee_R_Joint: limit lower=-1.75192 upper=0.523599 effort=4.5 velocity=15 -> lower=-1.75192 upper=0.523599 effort=4.5 velocity=33.5
- joint thigh_L_Joint: limit lower=-0.593412 upper=1.88496 effort=4.5 velocity=15.0 -> lower=-0.593412 upper=1.88496 effort=4.5 velocity=33.5
- joint thigh_R_Joint: limit lower=-1.88496 upper=0.593412 effort=4.5 velocity=15.0 -> lower=-1.88496 upper=0.593412 effort=4.5 velocity=33.5
- joint wheel_L_Joint: limit lower=-1000000 upper=1000000 effort=2.5 velocity=40 -> lower=-1000000 upper=1000000 effort=2.5 velocity=33.5
- joint wheel_R_Joint: limit lower=-1000000 upper=1000000 effort=2.5 velocity=40 -> lower=-1000000 upper=1000000 effort=2.5 velocity=33.5
