Commit message: feat : goat_description urdf update

File: Realworld/src/goat_description/urdf/WF_GOAT.urdf (robot description, URDF)
Before this commit: robot wheel_TRON, 9 links, 8 joints
Links:
- link base_Link: mass 9.585 -> 2.818; geometry collision box size=0.27 0.26 0.19; visual mesh filename=../meshes/base_Link.STL
- link calf_L_Link: mass 1.49 -> 0.287; geometry collision cylinder length=0.26 radius=0.015; visual mesh filename=../meshes/calf_L_Link.STL
- link calf_R_Link: mass 1.49 -> 0.287; geometry collision cylinder length=0.26 radius=0.015; visual mesh filename=../meshes/calf_R_Link.STL
- link hip_L_Link: mass 1.469 -> 0.32; geometry collision cylinder length=0.05 radius=0.05; visual mesh filename=../meshes/hip_L_Link.STL
- link hip_R_Link: mass 1.469 -> 0.32; geometry collision cylinder length=0.05 radius=0.05; visual mesh filename=../meshes/hip_R_Link.STL
- link thigh_L_Link: mass 2.3 -> 0.429; geometry collision cylinder length=0.15 radius=0.035; visual mesh filename=../meshes/thigh_L_Link.STL
- link thigh_R_Link: mass 2.30 -> 0.429; geometry collision cylinder length=0.15 radius=0.035; visual mesh filename=../meshes/thigh_R_Link.STL
- link wheel_L_Link: mass 1.08 -> 0.212; geometry collision cylinder length=0.05 radius=0.127; visual mesh filename=../meshes/wheel_L_Link.STL
- link wheel_R_Link: mass 1.08 -> 0.212; geometry collision cylinder length=0.05 radius=0.127; visual mesh filename=../meshes/wheel_R_Link.STL

Commit message: fix : ros2 urdf file location

File: Realworld/src/goat_description/urdf/WF_GOAT.urdf (robot description, URDF)
Before this commit: robot wheel_TRON, 9 links, 8 joints
Links:
- link base_Link: geometry collision box size=0.27 0.26 0.19; visual mesh filename=package://goat_description/meshes/base_Link.stl scale=1 1 1
- link calf_L_Link: geometry collision cylinder length=0.26 radius=0.015; visual mesh filename=package://goat_description/meshes/calf_L_Link.stl scale=1 1 1
- link calf_R_Link: geometry collision cylinder length=0.26 radius=0.015; visual mesh filename=package://goat_description/meshes/calf_R_Link.stl scale=1 1 1
- link hip_L_Link: geometry collision cylinder length=0.05 radius=0.05; visual mesh filename=package://goat_description/meshes/hip_L_Link.stl scale=1 1 1
- link hip_R_Link: geometry collision cylinder length=0.05 radius=0.05; visual mesh filename=package://goat_description/meshes/hip_R_Link.stl scale=1 1 1
- link thigh_L_Link: geometry collision cylinder length=0.15 radius=0.035; visual mesh filename=package://goat_description/meshes/thigh_L_Link.stl scale=1 1 1
- link thigh_R_Link: geometry collision cylinder length=0.15 radius=0.035; visual mesh filename=package://goat_description/meshes/thigh_R_Link.stl scale=1 1 1
- link wheel_L_Link: geometry collision cylinder length=0.05 radius=0.127; visual mesh filename=package://goat_description/meshes/wheel_L_Link.stl scale=1 1 1
- link wheel_R_Link: geometry collision cylinder length=0.05 radius=0.127; visual mesh filename=package://goat_description/meshes/wheel_R_Link.stl scale=1 1 1

Commit message: feat: collision region setting

File: Realworld/src/goat_description/urdf/WF_GOAT.urdf (robot description, URDF)
Before this commit: robot wheel_TRON, 9 links, 8 joints
Links:
- link base_Link: geometry collision box size=0.214 0.200 0.190; visual mesh filename=package://goat_description/meshes/base_Link.stl scale=1 1 1
- link calf_L_Link: geometry collision cylinder length=233E-03 radius=32.5E-03; visual mesh filename=package://goat_description/meshes/calf_L_Link.stl scale=1 1 1
- link calf_R_Link: geometry collision cylinder length=233E-03 radius=32.5E-03; visual mesh filename=package://goat_description/meshes/calf_R_Link.stl scale=1 1 1
- link hip_L_Link: geometry collision cylinder length=48E-03 radius=43.5E-03; visual mesh filename=package://goat_description/meshes/hip_L_Link.stl scale=1 1 1
- link hip_R_Link: geometry collision cylinder length=48E-03 radius=43.5E-03; visual mesh filename=package://goat_description/meshes/hip_R_Link.stl scale=1 1 1
- link thigh_L_Link: geometry collision cylinder length=266E-03 radius=41E-03; visual mesh filename=package://goat_description/meshes/thigh_L_Link.stl scale=1 1 1
- link thigh_R_Link: geometry collision cylinder length=266E-03 radius=41E-03; visual mesh filename=package://goat_description/meshes/thigh_R_Link.stl scale=1 1 1
- link wheel_L_Link: geometry collision cylinder length=32E-03 radius=73E-03; visual mesh filename=package://goat_description/meshes/wheel_L_Link.stl scale=1 1 1
- link wheel_R_Link: geometry collision cylinder length=32E-03 radius=73E-03; visual mesh filename=package://goat_description/meshes/wheel_R_Link.stl scale=1 1 1

Commit message: remove motor_state_interface

File: Realworld/src/goat_description/urdf/WF_GOAT.urdf (robot description, URDF)
Before this commit: robot wheel_TRON, 9 links, 8 joints
Joints:
- joint wheel_L_Joint: axis 0 -1 0 -> 0 1 0
- joint wheel_R_Joint: axis 0 1 0 -> 0 -1 0

Commit message: merge

File: Realworld/src/goat_description/urdf/WF_GOAT.urdf (robot description, URDF)
Before this commit: robot wheel_TRON, 9 links, 8 joints
Links:
- link base_Link: mass 9.585 -> 2.818; geometry collision box size=0.214 0.200 0.190; visual mesh filename=package://goat_description/meshes/base_Link.stl scale=1 1 1
- link calf_L_Link: mass 1.49 -> 0.287; geometry collision cylinder length=233E-03 radius=32.5E-03; visual mesh filename=package://goat_description/meshes/calf_L_Link.stl scale=1 1 1
- link calf_R_Link: mass 1.49 -> 0.287; geometry collision cylinder length=233E-03 radius=32.5E-03; visual mesh filename=package://goat_description/meshes/calf_R_Link.stl scale=1 1 1
- link hip_L_Link: mass 1.469 -> 0.32; geometry collision cylinder length=48E-03 radius=43.5E-03; visual mesh filename=package://goat_description/meshes/hip_L_Link.stl scale=1 1 1
- link hip_R_Link: mass 1.469 -> 0.32; geometry collision cylinder length=48E-03 radius=43.5E-03; visual mesh filename=package://goat_description/meshes/hip_R_Link.stl scale=1 1 1
- link thigh_L_Link: mass 2.3 -> 0.429; geometry collision cylinder length=266E-03 radius=41E-03; visual mesh filename=package://goat_description/meshes/thigh_L_Link.stl scale=1 1 1
- link thigh_R_Link: mass 2.30 -> 0.429; geometry collision cylinder length=266E-03 radius=41E-03; visual mesh filename=package://goat_description/meshes/thigh_R_Link.stl scale=1 1 1
- link wheel_L_Link: mass 1.08 -> 0.212; geometry collision cylinder length=32E-03 radius=73E-03; visual mesh filename=package://goat_description/meshes/wheel_L_Link.stl scale=1 1 1
- link wheel_R_Link: mass 1.08 -> 0.212; geometry collision cylinder length=32E-03 radius=73E-03; visual mesh filename=package://goat_description/meshes/wheel_R_Link.stl scale=1 1 1
Joints:
- joint wheel_L_Joint: axis 0 -1 0 -> 0 1 0
- joint wheel_R_Joint: axis 0 1 0 -> 0 -1 0

Commit message: visualization imu

File: Realworld/src/goat_description/urdf/WF_GOAT.urdf (robot description, URDF)
Before this commit: robot wheel_TRON, 9 links, 8 joints
Links:
- added link imu_link
Joints:
- added joint imu_joint: type fixed, parent base_Link, child imu_link, origin xyz=0 0 0.1 rpy=0 0 0

Commit message: change joint limit cfg

File: Realworld/src/goat_description/urdf/WF_GOAT.urdf (robot description, URDF)
Before this commit: robot wheel_TRON, 9 links, 8 joints
Joints:
- joint hip_L_Joint: limit lower=-2.05949 upper=1.09956 effort=4.5 velocity=15.0 -> lower=-1.22173 upper=0.750492 effort=4.5 velocity=15.0
- joint hip_R_Joint: limit lower=-1.09956 upper=2.05949 effort=4.5 velocity=15.0 -> lower=-0.750492 upper=1.22173 effort=4.5 velocity=15.0
- joint knee_L_Joint: limit lower=0.0 upper=1.75192 effort=4.5 velocity=15 -> lower=0.0 upper=2.30383 effort=4.5 velocity=15
- joint knee_R_Joint: limit lower=-1.75192 upper=0.0 effort=4.5 velocity=15 -> lower=-2.30383 upper=0.0 effort=4.5 velocity=15
- joint thigh_L_Joint: limit lower=-0.593412 upper=1.88496 effort=4.5 velocity=15.0 -> lower=-0.261799 upper=2.05949 effort=4.5 velocity=15.0
- joint thigh_R_Joint: limit lower=-1.88496 upper=0.593412 effort=4.5 velocity=15.0 -> lower=-2.05949 upper=0.261799 effort=4.5 velocity=15.0

File: src/lib/assets/GOAT/WF_GOAT/urdf/WF_GOAT.urdf (robot description, URDF)
Before this commit: robot wheel_GOAT, 9 links, 8 joints
Joints:
- joint hip_L_Joint: limit lower=-2.05949 upper=1.09956 effort=4.5 velocity=33.5 -> lower=-1.22173 upper=0.750492 effort=4.5 velocity=15.0
- joint hip_R_Joint: limit lower=-1.09956 upper=2.05949 effort=4.5 velocity=33.5 -> lower=-0.750492 upper=1.22173 effort=4.5 velocity=15.0
- joint knee_L_Joint: limit lower=-0.523599 upper=1.75192 effort=4.5 velocity=33.5 -> lower=0.0 upper=2.30383 effort=4.5 velocity=15
- joint knee_R_Joint: limit lower=-1.75192 upper=0.523599 effort=4.5 velocity=33.5 -> lower=-2.30383 upper=0.0 effort=4.5 velocity=15
- joint thigh_L_Joint: limit lower=-0.593412 upper=1.88496 effort=4.5 velocity=33.5 -> lower=-0.261799 upper=2.05949 effort=4.5 velocity=15.0
- joint thigh_R_Joint: limit lower=-1.88496 upper=0.593412 effort=4.5 velocity=33.5 -> lower=-2.05949 upper=0.261799 effort=4.5 velocity=15.0
- joint wheel_L_Joint: limit lower=-1000000 upper=1000000 effort=2.5 velocity=33.5 -> lower=-1000000 upper=1000000 effort=2.5 velocity=40
- joint wheel_R_Joint: limit lower=-1000000 upper=1000000 effort=2.5 velocity=33.5 -> lower=-1000000 upper=1000000 effort=2.5 velocity=40

Commit message: update mass

File: Realworld/src/goat_description/urdf/WF_GOAT.urdf (robot description, URDF)
Before this commit: robot wheel_GOAT, 10 links, 9 joints
Links:
- removed link imu_link
- link base_Link: mass 2.818 -> 3.075; geometry collision box size=0.214 0.200 0.190; visual mesh filename=../meshes/base_Link.stl
- link calf_L_Link: mass 0.287 -> 0.321; geometry collision cylinder length=233E-03 radius=32.5E-03; visual mesh filename=../meshes/calf_L_Link.stl
- link calf_R_Link: mass 0.287 -> 0.321; geometry collision cylinder length=233E-03 radius=32.5E-03; visual mesh filename=../meshes/calf_R_Link.stl
- link hip_L_Link: mass 0.32 -> 0.316; geometry collision cylinder length=48E-03 radius=43.5E-03; visual mesh filename=../meshes/hip_L_Link.stl
- link hip_R_Link: mass 0.32 -> 0.316; geometry collision cylinder length=48E-03 radius=43.5E-03; visual mesh filename=../meshes/hip_R_Link.stl
- link thigh_L_Link: mass 0.429 -> 0.473; geometry collision cylinder length=266E-03 radius=41E-03; visual mesh filename=../meshes/thigh_L_Link.stl
- link thigh_R_Link: mass 0.429 -> 0.473; geometry collision cylinder length=266E-03 radius=41E-03; visual mesh filename=../meshes/thigh_R_Link.stl
- link wheel_L_Link: mass 0.212 -> 0.238; geometry collision cylinder length=32E-03 radius=72.75E-03; visual mesh filename=../meshes/wheel_L_Link.stl
- link wheel_R_Link: mass 0.212 -> 0.238; geometry collision cylinder length=32E-03 radius=72.75E-03; visual mesh filename=../meshes/wheel_R_Link.stl
Joints:
- removed joint imu_joint

File: src/lib/assets/GOAT/WF_GOAT/urdf/WF_GOAT.urdf (robot description, URDF)
Before this commit: robot wheel_GOAT, 10 links, 9 joints
Links:
- removed link imu_link
- link base_Link: mass 2.818 -> 3.075
- link calf_L_Link: mass 0.287 -> 0.321
- link calf_R_Link: mass 0.287 -> 0.321
- link hip_L_Link: mass 0.32 -> 0.316
- link hip_R_Link: mass 0.32 -> 0.316
- link thigh_L_Link: mass 0.429 -> 0.473
- link thigh_R_Link: mass 0.429 -> 0.473
- link wheel_L_Link: mass 0.212 -> 0.238
- link wheel_R_Link: mass 0.212 -> 0.238
Joints:
- removed joint imu_joint

Commit message: import error

File: Realworld/src/goat_description/urdf/WF_GOAT.urdf (robot description, URDF)
Before this commit: robot wheel_GOAT, 10 links, 9 joints
Links:
- link base_Link: geometry collision box size=0.214 0.200 0.190; visual mesh filename=package://goat_description/meshes/base_Link.stl
- link calf_L_Link: geometry collision cylinder length=233E-03 radius=32.5E-03; visual mesh filename=package://goat_description/meshes/calf_L_Link.stl
- link calf_R_Link: geometry collision cylinder length=233E-03 radius=32.5E-03; visual mesh filename=package://goat_description/meshes/calf_R_Link.stl
- link hip_L_Link: geometry collision cylinder length=48E-03 radius=43.5E-03; visual mesh filename=package://goat_description/meshes/hip_L_Link.stl
- link hip_R_Link: geometry collision cylinder length=48E-03 radius=43.5E-03; visual mesh filename=package://goat_description/meshes/hip_R_Link.stl
- link thigh_L_Link: geometry collision cylinder length=266E-03 radius=41E-03; visual mesh filename=package://goat_description/meshes/thigh_L_Link.stl
- link thigh_R_Link: geometry collision cylinder length=266E-03 radius=41E-03; visual mesh filename=package://goat_description/meshes/thigh_R_Link.stl
- link wheel_L_Link: geometry collision cylinder length=32E-03 radius=72.75E-03; visual mesh filename=package://goat_description/meshes/wheel_L_Link.stl
- link wheel_R_Link: geometry collision cylinder length=32E-03 radius=72.75E-03; visual mesh filename=package://goat_description/meshes/wheel_R_Link.stl
