Commit message: URDF

File: Realworld/src/goat_description/urdf/WF_GOAT.urdf (robot description, URDF)
Before this commit: robot wheel_GOAT, 10 links, 9 joints
Links:
- link hip_L_Link: geometry collision cylinder length=135E-03 radius=42E-03; visual mesh filename=package://goat_description/meshes/hip_L_Link.stl
- link hip_R_Link: geometry collision cylinder length=135E-03 radius=42E-03; visual mesh filename=package://goat_description/meshes/hip_R_Link.stl
- link thigh_L_Link: geometry collision box size=0.09 0.05 0.145; visual mesh filename=package://goat_description/meshes/thigh_L_Link.stl
- link thigh_R_Link: geometry collision box size=0.09 0.05 0.145; visual mesh filename=package://goat_description/meshes/thigh_R_Link.stl

Commit message: Hw test

File: Realworld/src/goat_description/urdf/WF_GOAT.urdf (robot description, URDF)
Before this commit: robot wheel_GOAT, 10 links, 9 joints
Links:
- link base_Link: mass 2.818 -> 3.119
- link calf_L_Link: mass 0.299 -> 0.326
- link calf_R_Link: mass 0.299 -> 0.327
- link hip_L_Link: mass 0.32 -> 0.316
- link hip_R_Link: mass 0.32 -> 0.322
- link thigh_L_Link: mass 0.483 -> 0.496
- link thigh_R_Link: mass 0.483 -> 0.495
- link wheel_L_Link: mass 0.212 -> 0.239
- link wheel_R_Link: mass 0.212 -> 0.217
Joints:
- joint hip_L_Joint: limit lower=-2.05949 upper=1.09956 effort=4.5 velocity=33.5 -> lower=-1.7453 upper=1.0123 effort=4.5 velocity=33.5
- joint hip_R_Joint: limit lower=-1.09956 upper=2.05949 effort=4.5 velocity=33.5 -> lower=-1.0123 upper=1.7453 effort=4.5 velocity=33.5
- joint knee_L_Joint: limit lower=-0.523599 upper=1.75192 effort=4.5 velocity=33.5 -> lower=-0.523599 upper=2.3387 effort=4.5 velocity=33.5
- joint knee_R_Joint: limit lower=-1.75192 upper=0.523599 effort=4.5 velocity=33.5 -> lower=-2.3387 upper=0.523599 effort=4.5 velocity=33.5
- joint thigh_L_Joint: limit lower=-0.593412 upper=1.88496 effort=4.5 velocity=33.5 -> lower=-0.3840 upper=2.0071 effort=4.5 velocity=33.5
- joint thigh_R_Joint: limit lower=-1.88496 upper=0.593412 effort=4.5 velocity=33.5 -> lower=-2.0071 upper=0.3840 effort=4.5 velocity=33.5

Commit message: .

File: Realworld/src/goat_description/urdf/WF_GOAT.urdf (robot description, URDF)
Before this commit: robot wheel_GOAT, 10 links, 9 joints
Links:
- link wheel_L_Link: mass 0.239 -> 0.985; geometry collision cylinder length=0.05 radius=0.1; visual mesh filename=package://goat_description//meshes/New_wheel_L_Link.stl
- link wheel_R_Link: mass 0.217 -> 0.985; geometry collision cylinder length=0.05 radius=0.1; visual mesh filename=package://goat_description/meshes/New_wheel_R_Link.stl

Commit message: .

File: Realworld/src/goat_description/urdf/WF_GOAT.urdf (robot description, URDF)
Before this commit: robot wheel_GOAT, 10 links, 9 joints
Links:
- link wheel_L_Link: mass 0.985 -> 0.239; geometry collision cylinder length=32E-03 radius=72.75E-03; visual mesh filename=package://goat_description/meshes/wheel_L_Link.stl
- link wheel_R_Link: mass 0.985 -> 0.217; geometry collision cylinder length=32E-03 radius=72.75E-03; visual mesh filename=package://goat_description/meshes/wheel_R_Link.stl

Commit message: URDF

File: Realworld/src/goat_description/urdf/WF_GOAT.urdf (robot description, URDF)
Before this commit: robot wheel_GOAT, 10 links, 9 joints
Links:
- link base_Link: mass 3.119 -> 3.153308; geometry collision box size=0.07 0.25 0.08; collision box size=0.214 0.200 0.190
- link calf_L_Link: mass 0.326 -> 0.303
- link calf_R_Link: mass 0.327 -> 0.303
- link hip_L_Link: mass 0.316 -> 0.319
- link hip_R_Link: mass 0.322 -> 0.319
- link thigh_L_Link: mass 0.496 -> 0.483216
- link thigh_R_Link: mass 0.495 -> 0.483216
- link wheel_L_Link: mass 0.239 -> 0.985; geometry collision cylinder length=0.05 radius=0.1; visual mesh filename=package://goat_description/meshes/New_wheel_L_Link.stl
- link wheel_R_Link: mass 0.217 -> 0.985; geometry collision cylinder length=0.05 radius=0.1; visual mesh filename=package://goat_description/meshes/New_wheel_R_Link.stl
Joints:
- joint hip_L_Joint: origin xyz=38.386E-03 94.233E-03 -152.597E-03 rpy=0 0 0 -> xyz=49.579E-03 96.336E-03 -87.088E-03 rpy=0 0 0
- joint hip_R_Joint: origin xyz=38.386E-03 -94.233E-03 -152.597E-03 rpy=0 0 0 -> xyz=49.579E-03 -96.336E-03 -87.088E-03 rpy=0 0 0

Commit message: .

File: Realworld/src/goat_description/urdf/WF_GOAT.urdf (robot description, URDF)
Before this commit: robot wheel_GOAT, 10 links, 9 joints
Links:
- link wheel_L_Link: mass 0.985 -> 0.220; geometry collision cylinder length=7E-03 radius=72.75E-03; visual mesh filename=package://goat_description/meshes/wheel_L_Link.stl
- link wheel_R_Link: mass 0.985 -> 0.220; geometry collision cylinder length=7E-03 radius=72.75E-03; visual mesh filename=package://goat_description/meshes/wheel_R_Link.stl

Commit message: URDF Ssibal

File: Realworld/src/goat_description/urdf/WF_GOAT.urdf (robot description, URDF)
Before this commit: robot wheel_GOAT, 10 links, 9 joints
Links:
- link wheel_L_Link: mass 0.220 -> 0.985; geometry collision cylinder length=0.05 radius=0.1; visual mesh filename=package://goat_description/meshes/New_wheel_L_Link.stl
- link wheel_R_Link: mass 0.220 -> 0.985; geometry collision cylinder length=0.05 radius=0.1; visual mesh filename=package://goat_description/meshes/New_wheel_R_Link.stl

Commit message: urdf update

File: Realworld/src/goat_description/urdf/WF_GOAT.urdf (robot description, URDF)
Before this commit: robot wheel_GOAT, 10 links, 9 joints
Links:
- link base_Link: mass 3.119 -> 3.153308; geometry collision box size=0.07 0.25 0.08; collision box size=0.214 0.200 0.190
- link calf_L_Link: mass 0.326 -> 0.303; geometry collision cylinder length=233E-03 radius=32.5E-03; visual mesh filename=../meshes/calf_L_Link.stl
- link calf_R_Link: mass 0.327 -> 0.303; geometry collision cylinder length=233E-03 radius=32.5E-03; visual mesh filename=../meshes/calf_R_Link.stl
- link hip_L_Link: mass 0.316 -> 0.319; geometry collision cylinder length=135E-03 radius=42E-03; visual mesh filename=../meshes/hip_L_Link.stl
- link hip_R_Link: mass 0.322 -> 0.319; geometry collision cylinder length=135E-03 radius=42E-03; visual mesh filename=../meshes/hip_R_Link.stl
- link thigh_L_Link: mass 0.496 -> 0.483216; geometry collision box size=0.09 0.05 0.145; visual mesh filename=../meshes/thigh_L_Link.stl
- link thigh_R_Link: mass 0.495 -> 0.483216; geometry collision box size=0.09 0.05 0.145; visual mesh filename=../meshes/thigh_R_Link.stl
- link wheel_L_Link: mass 0.239 -> 0.985; geometry collision cylinder length=0.05 radius=0.1; visual mesh filename=../meshes/BF_wheel_L_Link.stl
- link wheel_R_Link: mass 0.217 -> 0.985; geometry collision cylinder length=0.05 radius=0.1; visual mesh filename=../meshes/BF_wheel_R_Link.stl
Joints:
- joint hip_L_Joint: origin xyz=38.386E-03 94.233E-03 -152.597E-03 rpy=0 0 0 -> xyz=49.579E-03 96.336E-03 -87.088E-03 rpy=0 0 0
- joint hip_R_Joint: origin xyz=38.386E-03 -94.233E-03 -152.597E-03 rpy=0 0 0 -> xyz=49.579E-03 -96.336E-03 -87.088E-03 rpy=0 0 0
- joint knee_L_Joint: limit lower=-0.523599 upper=2.3387 effort=4.5 velocity=33.5 -> lower=-0.523599 upper=2.3387 effort=9.0 velocity=33.5
- joint knee_R_Joint: limit lower=-2.3387 upper=0.523599 effort=4.5 velocity=33.5 -> lower=-2.3387 upper=0.523599 effort=9.0 velocity=33.5

Commit message: .

File: Realworld/src/goat_description/urdf/WF_GOAT.urdf (robot description, URDF)
Before this commit: robot wheel_GOAT, 10 links, 9 joints
Links:
- link hip_L_Link: mass 0.319 -> 0.326
- link hip_R_Link: mass 0.319 -> 0.326
Joints:
- joint hip_L_Joint: origin xyz=49.579E-03 96.336E-03 -87.088E-03 rpy=0 0 0 -> xyz=51.079E-03 96.336E-03 -87.088E-03 rpy=0 0 0
- joint hip_R_Joint: origin xyz=49.579E-03 -96.336E-03 -87.088E-03 rpy=0 0 0 -> xyz=51.079E-03 -96.336E-03 -87.088E-03 rpy=0 0 0

Commit message: .

File: Realworld/src/goat_description/urdf/WF_GOAT.urdf (robot description, URDF)
Before this commit: robot wheel_GOAT, 10 links, 9 joints
Links:
- link base_Link: geometry collision box size=0.214 0.200 0.190; visual mesh filename=../meshes/base_Link.stl

Commit message: .

File: Realworld/src/goat_description/urdf/WF_GOAT.urdf (robot description, URDF)
Before this commit: robot wheel_GOAT, 10 links, 9 joints
Joints:
- joint hip_L_Joint: type revolute -> fixed
- joint hip_R_Joint: type revolute -> fixed
